Commit message: updating transforms
added kinect to urdf and updated the transforms to be more accurate

File: mrcrabs.urdf (robot description, URDF)
Before this commit: robot mrcrabs, 6 links, 5 joints
Links:
- added link kinect; visual box size=${kinect_size}
Joints:
- added joint kinect_rotate: type revolute, parent base_link, child kinect, origin xyz=${kinect_xoff} 0 ${kinect_zoff}, axis 0 1 0, limit lower=0.471239 upper=0.471239 effort=1000.0 velocity=0.1
- joint back_sonar_joint: origin xyz=-${sonar_xoff} 0 ${sonar_zoff} -> xyz=-${sonar_xoff} 0 ${sonar_zoff} rpy=0 0 -1.57075
- joint front_sonar_joint: origin xyz=${sonar_xoff} 0 ${sonar_zoff} -> xyz=${sonar_xoff} 0 ${sonar_zoff} rpy=0 0 1.57075

Commit message: updating transforms
added kinect to urdf and updated the transforms to be more accurate

File: mrcrabs.urdf (robot description, URDF)
Before this commit: robot mrcrabs, 6 links, 5 joints
Links:
- added link bl_wheel; visual cylinder length=${wheel_width} radius=${wheel_radius}
- added link br_wheel; visual cylinder length=${wheel_width} radius=${wheel_radius}
- added link fl_wheel; visual cylinder length=${wheel_width} radius=${wheel_radius}
- added link fr_wheel; visual cylinder length=${wheel_width} radius=${wheel_radius}
- added link kinect; visual box size=${kinect_size}
Joints:
- added joint bl_wheel_cont: type continuous, parent base_link, child bl_wheel, origin xyz=-${wheel_xoff} -${wheel_ygap} ${wheel_zoff}, axis 0 1 0
- added joint br_wheel_cont: type continuous, parent base_link, child br_wheel, origin xyz=-${wheel_xoff} ${wheel_ygap} ${wheel_zoff}, axis 0 1 0
- added joint fl_wheel_cont: type continuous, parent base_link, child fl_wheel, origin xyz=${wheel_xoff} -${wheel_ygap} ${wheel_zoff}, axis 0 1 0
- added joint fr_wheel_cont: type continuous, parent base_link, child fr_wheel, origin xyz=${wheel_xoff} ${wheel_ygap} ${wheel_zoff}, axis 0 1 0
- added joint kinect_rotate: type revolute, parent base_link, child kinect, origin xyz=${kinect_xoff} 0 ${kinect_zoff}, axis 0 1 0, limit lower=-0.471239 upper=0.471239 effort=1000.0 velocity=0.1
- joint back_sonar_joint: origin xyz=-${sonar_xoff} 0 ${sonar_zoff} -> xyz=-${sonar_xoff} 0 ${sonar_zoff} rpy=0 0 -1.57075
- joint front_sonar_joint: origin xyz=${sonar_xoff} 0 ${sonar_zoff} -> xyz=${sonar_xoff} 0 ${sonar_zoff} rpy=0 0 1.57075
